File: arduino_test/block_sch/block_sch.kicad_sch (KiCad schematic)
At the start: 1 part

Commit message: Draw basic inital schematic
Other:
- note added: "6-pin ISCP header MISO/MOSI/SCK/ RESET/GND/VCC VCC not connected"
- note added: "OSC 32.768 kHz, Quartz"
- note added: "UART1"
- note added: "USB 2.0 to UART bridge"
- note removed: "5 pin debug header VCC floating"
- note removed: "6-pin ISCP header MISO/MOSI/SCK/ RESET/GND/VCC VCC floating"
- note removed: "USART1"
- note removed: "USART2"
- note removed: "USB 2.0 to USART bridge"
Changed lines of the file:
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@@
-	(bus
-		(pts
-			(xy 181.61 115.57) (xy 187.96 115.57)
-		)
-		(stroke
-			(width 0)
-			(type default)
-		)
-	)
 	(bus
 		(pts
@@
 		(pts
 			(xy 265.43 68.58) (xy 265.43 74.93)
+		)
+		(stroke
+			(width 0)
+			(type default)
+		)
+	)
+	(bus
+		(pts
+			(xy 265.43 52.07) (xy 265.43 58.42)
 		)
 		(stroke
@@
 	)
 	(rectangle
-		(start 187.96 110.49)
-		(end 212.09 120.65)
+		(start 252.73 41.656)
+		(end 278.13 51.816)
 		(stroke
 			(width 0)
@@
 		)
 	)
+	(text "OSC 32.768 kHz,\nQuartz"
+		(exclude_from_sim no)
+		(at 265.43 46.99 0)
+		(effects
+			(font
+				(size 1.397 1.397)
+			)
+		)
+	)
 	(text "GPO"
 		(exclude_from_sim no)
@@
 		)
 	)
-	(text "6-pin ISCP header\nMISO/MOSI/SCK/\nRESET/GND/VCC\nVCC floating"
+	(text "6-pin ISCP header\nMISO/MOSI/SCK/\nRESET/GND/VCC\nVCC not connected"
 		(exclude_from_sim no)
 		(at 237.49 105.41 0)
@@
 		)
 	)
-	(text "5 pin debug header\nVCC floating"
-		(exclude_from_sim no)
-		(at 200.152 115.824 0)
-		(effects
-			(font
-				(size 1.397 1.397)
-			)
-		)
-	)
 	(text "I2C"
 		(exclude_from_sim no)
@@
 		)
 	)
-	(text "USART2"
-		(exclude_from_sim no)
-		(at 176.784 115.824 0)
-		(effects
-			(font
-				(size 1.397 1.397)
-			)
-		)
-	)
 	(text "MCU\nATMega328p"
 		(exclude_from_sim no)
@@
 		)
 	)
-	(text "USART1"
+	(text "UART1"
 		(exclude_from_sim no)
 		(at 149.098 67.818 0)
@@
 		)
 	)
-	(text "USB 2.0 to \nUSART bridge"
+	(text "USB 2.0 to \nUART bridge"
 		(exclude_from_sim no)
 		(at 84.582 67.564 0)
