File: ICSP.kicad_sch (KiCad schematic)
At the start: 6 parts, among them J4 Conn_02x03_Counter_Clockwise, U10 74LVC2G125DCTRE4, U11 SN74LV1T34DBV, U12 74LVC1G04, U9 74LVC2G125DCTRE4

Commit message: Touchup schematics
Parts:
- added C10, C15, C16, C9: 0.1, symbol Device:C
- added D3, D4, D5, D6, D7: ESD131-B1-W0201, Diode_SMD:Infineon_SG-WLL-2-3_0.58x0.28_P0.36mm, symbol Diode:ESD131-B1-W0201
Connections:
- net 5V: now also C15.1, D3.1 (A1)
- net GND: now also C10.2, C15.2, C16.2, C9.2, D3.2 (A2), D4.2 (A2), D5.2 (A2), D6.2 (A2), D7.2 (A2)
- net MISO 5V: now also D7.1 (A1)
- net MOSI 5V: now also D4.1 (A1)
- net RESET 5V: now also D6.1 (A1)
- net SCK 5V: now also D5.1 (A1)
- net VCC: now also C10.1, C16.1, C9.1
Other:
- note added: "Connection for 5V ICS programmer"
- note removed: "TODO: Replace with 1x logic"
- moved on the sheet: R28, U10, U11, U12, U9

Commit message: viskasin kõik ühele lehele.
Parts:
- removed C10, C15, C16, C9: 0.1, symbol Device:C
- removed D3, D4, D5, D6, D7: ESD131-B1-W0201, Diode_SMD:Infineon_SG-WLL-2-3_0.58x0.28_P0.36mm, symbol Diode:ESD131-B1-W0201
- removed J4: Conn_02x03_Counter_Clockwise, symbol Connector_Generic:Conn_02x03_Counter_Clockwise
- removed R28: 10k, symbol Device:R
- removed U10, U9: 74LVC2G125DCTRE4, DCT8, symbol 2024-11-19_12-34-20:74LVC2G125DCTRE4
- removed U11: SN74LV1T34DBV, Package_TO_SOT_SMD:SOT-23-5, symbol Logic_LevelTranslator:SN74LV1T34DBV
- removed U12: 74LVC1G04, symbol 74xGxx:74LVC1G04
Connections:
- no-connect marks 1 -> 0
Other:
- note removed: "Connection for 5V ICS programmer"
