File: MPU-6050.kicad_sch (KiCad schematic)
At the start: 5 parts, among them U2 MPU-6050

Commit message: Touchup schematics
Other:
- note added: "Accelerometer + gryoscope"
Changed lines of the file:
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@@
+		)
+	)
+	(text "Accelerometer + gryoscope"
+		(exclude_from_sim no)
+		(at 41.91 16.51 0)
+		(effects
+			(font
+				(size 1.27 1.27)
+			)
 		)
 	)
 	(text "All capacitors are +-10%"
 		(exclude_from_sim no)
-		(at 42.418 17.272 0)
+		(at 42.164 18.796 0)
 		(effects
 			(font

Commit message: viskasin kõik ühele lehele.
Parts:
- removed C3: 10n, 4V, symbol Device:C
- removed C4: 0.1u, 4V, symbol Device:C
- removed C5: 0.1u, 2V, symbol Device:C
- removed C6: 2.2n, 50V, symbol Device:C
- removed U2: MPU-6050, Sensor_Motion:InvenSense_QFN-24_4x4mm_P0.5mm, symbol Sensor_Motion:MPU-6050
Connections:
- no-connect marks 3 -> 0
Other:
- note removed: "Accelerometer + gryoscope"
- note removed: "All capacitors are +-10%"
