File: plokkskeem.kicad_sch (KiCad schematic)
At the start: 6 parts, among them U4 ATmega328P-A, Y1 10MHz

Commit message: Draw basic inital schematic
Parts:
- added D1: LED, symbol Device:LED
- added R1, R2, R29, R4, R5, R8, R9: 10k, symbol Device:R
- added R19: 30k, symbol Device:R
- added R3: 1k7, symbol Device:R
- renumbered R3 to R6, R4 to R7, U4 to U1
Connections:
- net GND: now also D1.1 (K), R1.1, R2.1, R29.1
- net RESET: now also R9.2
- net SCL: now also R6.1; no longer R7.1
- net SDA: now also R7.2; no longer R6.1
- net SS: now also R8.1
- net VCC: now also R7.1, R4.2, R5.1, R8.2, R9.1; no longer R7.2
- net XTAL2: now reaches C2.1, U1.8 (XTAL2/PB7), Y1.1
- net XTAL1: now reaches C1.1, U1.7 (XTAL1/PB6), Y1.2
- net CTS: now reaches U1.1 (PD3)
- net at U1.19 (ADC6): now also R1.2
- net at U1.22 (ADC7): now also R2.2
- net VTEMP: now reaches U1.24 (PC1)
- net at U1.25 (PC2): now also R4.1
- net at U1.26 (PC3): now also R5.2
- net RTS: now reaches U1.32 (PD2)
- net LED: no longer names the net of U1.12 (PB0)
- net LED: now also R3.1
- net Patarei Analog renamed VBAT_DIV
- net VBAT_DIV: now also R19.1, R29.2
- net XCK renamed USB_DET
- new net: D1.2 (A), R3.2
- new net VBAT: R19.2
- no-connect marks 6 -> 1
Other:
- note added: "1.6 Vf, 1 mA"
- moved on the sheet: C1, C2, R6, R7, Y1

Commit message: Touchup schematics
Parts:
- added U18, U19: ESD321DPYR, DPY2_TEX, symbol 2024-11-26_15-40-10:ESD321DPYR
Connections:
- net GND: now also U18.2 (GND), U19.2 (GND)
- net SCL: now also U19.1 (IO)
- net SDA: now also U18.1 (IO)
Other:
- note added: "1.6 Vf, 1 mA, red"
- note added: "Needed due to traces being long potentially?"
- note removed: "1.6 Vf, 1 mA"

Commit message: viskasin kõik ühele lehele.
Parts:
- added C10, C15, C16, C9: 0.1, symbol Device:C
- added C11, C17, C8: 0.1u, symbol Device:C
- added C12: 2.2u, symbol Device:C
- added C13: 4.7u, symbol Device:C
- added C14: 10u, symbol Device:C
- added C3: 10n, 4V, symbol Device:C
- added C4: 0.1u, 4V, symbol Device:C
- added C5: 0.1u, 2V, symbol Device:C
- added C6: 2.2n, 50V, symbol Device:C
- added C7: 1u, symbol Device:C
- added D2, D3, D4, D5, D6, D7: ESD131-B1-W0201, Diode_SMD:Infineon_SG-WLL-2-3_0.58x0.28_P0.36mm, symbol Diode:ESD131-B1-W0201
- added J1: Micro_SD_Card, symbol Connector:Micro_SD_Card
- added J2: USB_C_Receptacle, symbol Connector:USB_C_Receptacle
- added J3, J5, J6: Conn_02x01, symbol Connector_Generic:Conn_02x01
- added J4: Conn_02x03_Counter_Clockwise, symbol Connector_Generic:Conn_02x03_Counter_Clockwise
- added L1: 10u, symbol Device:L
- added Q1, Q2: BS870, Package_TO_SOT_SMD:SOT-23, symbol Transistor_FET:BS870
- added R10: 30k, symbol Device:R
- added R11, R12: 5.1k, symbol Device:R
- added R13, R15, R22, R23, R24, R25, R26, R27, R28, R30: 10k, symbol Device:R
- added R14, R21: 1k, symbol Device:R
- added R16: 2k, symbol Device:R
- added R17: 36.5k, E48, symbol Device:R
- added R18: 953, E48, symbol Device:R
- added R20: 470, symbol Device:R
- added TH1, TH2: 10k, symbol Device:Thermistor_NTC
- added U10, U9: 74LVC2G125DCTRE4, DCT8, symbol 2024-11-19_12-34-20:74LVC2G125DCTRE4
- added U11: SN74LV1T34DBV, Package_TO_SOT_SMD:SOT-23-5, symbol Logic_LevelTranslator:SN74LV1T34DBV
- added U12: 74LVC1G04, symbol 74xGxx:74LVC1G04
- added U13: CP2102N-Axx-xQFN28, Package_DFN_QFN:QFN-28-1EP_5x5mm_P0.5mm_EP3.35x3.35mm, symbol Interface_USB:CP2102N-Axx-xQFN28
- added U2: MPU-6050, Sensor_Motion:InvenSense_QFN-24_4x4mm_P0.5mm, symbol Sensor_Motion:MPU-6050
- added U3: DS1307ZN+, Package_SO:SOIC-8_3.9x4.9mm_P1.27mm, symbol Timer_RTC:DS1307ZN+
- added U4, U5: ESD321DPYR, DPY2_TEX, symbol 2024-11-26_15-40-10:ESD321DPYR
- added U6: S-8261ABJMD-G3JT2G, IC6_S-8261ABJMD-G3JT2G_ABL, symbol 2024-11-21_09-28-04:S-8261ABJMD-G3JT2G
- added U7: BQ24032ARHLR, RHL0020A, symbol 2024-11-20_19-55-08:BQ24032ARHLR
- added U8: LTC3531EDD-PBF, DFN-8_DD_LIT, symbol 2024-11-21_16-20-21:LTC3531EDD-PBF
- added Y2: 32.768 kHz, symbol Device:Crystal
Connections:
- net CTS: now also U13.23 (~{CTS})
- net GND: now also C10.2, C11.2, C12.2, C13.2, C14.1, C15.2, C16.2, C17.2, C3.2, C4.2, C5.1, C6.2, C7.2, C8.1, C9.2, D2.2 (A2), D3.2 (A2), D4.2 (A2), D5.2 (A2), D6.2 (A2), D7.2 (A2), J1.6 (VSS), J1.9 (SHIELD), J2.A1 (GND), J2.A12 (GND), J2.B1 (GND), J2.B12 (GND), J2.S1 (SHIELD), J3.2 (Pin_2), J4.4 (Pin_4), J5.2 (Pin_2), Q2.2 (S), R11.2, R12.2, R14.1, R18.2, R22.2, R23.2, R24.2, R25.2, R26.2, R27.2, R28.2, R30.2, TH1.2, TH2.2, U10.4 (GND), U10.5 (2A), U11.3 (GND), U12.3 (GND), U13.29 (GND), U13.3 (GND), U2.1 (CLKIN), U2.11 (FSYNC), U2.18 (GND), U3.3 (VBAT), U3.4 (GND), U4.2 (GND), U5.2 (GND), U6.6 (VSS), U7.11 (VSS), U7.18 (ACPG_N), U7.2 (STAT1), U7.21 (EP), U7.3 (STAT2), U7.4 (AC), U8.3 (GND), U8.4 (*SHDN), U8.8 (PGND), U8.9 (EPAD), U9.4 (GND)
- net MISO: now also J1.7 (DAT0), U11.2 (A)
- net MOSI: now also J1.3 (CMD), U10.6 (1Y)
- net RESET: now also U9.3 (2Y)
- net RTS: now also U13.24 (~{RTS})
- net RXD: now also U13.25 (RXD)
- net SCK: now also J1.5 (CLK), U9.6 (1Y)
- net SCL: now also U2.23 (SCL), U3.6 (SCL)
- net SDA: now also U2.24 (SDA), U3.5 (SDA)
- net SD_CS: now also J1.2 (DAT3/CD)
- net TXD: now also U13.26 (TXD)
- net USB_DET: now also R13.2, U7.19 (USBPG_N)
- net VBAT: now also C11.1, J6.1 (Pin_1), R20.2, U7.5 (BAT), U7.6 (BAT)
- net VCC: now also C10.1, C13.1, C14.2, C15.1, C16.1, C17.1, C3.1, C4.1, J1.4 (VDD), R10.1, R13.1, R21.1, U10.8 (VCC), U12.5 (VCC), U13.6 (VDD), U13.7 (VREGIN), U2.13 (VDD), U2.8 (VLOGIC), U2.9 (AD0), U3.8 (VCC), U8.5 (FB), U8.6 (VOUT), U9.8 (VCC)
- net VTEMP: now also J3.1 (Pin_1), R10.2, TH1.1
- new net: Q1.1 (G), U6.1 (DO)
- new net: J6.2 (Pin_2), Q1.2 (S)
- new net: Q1.3 (D), Q2.3 (D), R16.1
- new net: R14.2, U7.10 (ISET1)
- new net: R23.1, U13.17 (RS485/GPIO.2)
- new net: R22.1, U13.19 (~{TXT}/GPIO.0)
- new net: R24.1, U13.22 (GPIO.4)
- new net: R16.2, U6.2 (VM)
- new net: R26.1, U13.18 (~{RXT}/GPIO.1)
- new net: R27.1, U13.16 (~{WAKEUP}/GPIO.3)
- new net: C5.2, U2.10 (REGOUT)
- new net: C6.1, U2.20 (CPOUT)
- new net: R25.1, U13.20 (GPIO.6)
- new net: U3.2 (X2), Y2.1
- new net: U3.1 (X1), Y2.2
- new net: R15.2, U7.8 (PSEL), U7.9 (CE)
- new net: C12.1, U7.15 (OUT), U7.16 (OUT), U7.17 (OUT), U8.2 (VIN)
- new net: Q2.1 (G), U6.3 (CO)
- new net: R20.1, U6.5 (VDD)
- new net: R17.1, U7.13 (DPPM)
- new net: R17.2, R18.1
- new net: R21.2, U13.9 (~{RST})
- new net: J2.A5 (CC1), R11.1
- new net: L1.1, U8.1 (SW1)
- new net: L1.2, U8.7 (SW2)
- new net: R30.1, U13.21 (GPIO.5)
- new net: J2.B5 (CC2), R12.1
- new net 5V: C9.1, D3.1 (A1), J4.6 (Pin_6), R28.1, U11.5 (VCC), U12.2
- new net CHR0: U13.15 (CHR0), U7.7 (ISET2)
- new net D+: J2.A6 (D+), J2.B6 (D+), U13.4 (D+), U5.1 (IO)
- new net D-: J2.A7 (D-), J2.B7 (D-), U13.5 (D-), U4.1 (IO)
- new net J3_EN: U10.1 (*1OE), U10.7 (*2OE), U12.4, U9.1 (*1OE), U9.7 (*2OE)
- new net MISO 5V: D7.1 (A1), J4.1 (Pin_1), U11.4 (Y)
- new net MOSI 5V: D4.1 (A1), J4.5 (Pin_5), U10.2 (1A)
- new net RESET 5V: D6.1 (A1), J4.3 (Pin_3), U9.5 (2A)
- new net SCK 5V: D5.1 (A1), J4.2 (Pin_2), U9.2 (1A)
- new net TS: J5.1 (Pin_1), TH2.1, U7.12 (TS)
- new net USB_LDO: R15.1, U7.1 (LDO), U7.14 (TMR)
- new net VBUS: C7.1, C8.2, D2.1 (A1), J2.A4 (VBUS), J2.A9 (VBUS), J2.B4 (VBUS), J2.B9 (VBUS), U13.8 (VBUS), U7.20 (USB)
- no-connect marks 1 -> 27
Other:
- note added: "103AT"
- note added: "37.4kOhm -> 3.74V dropout voltage"
- note added: "Accelerometer + gryoscope"
- note added: "All capacitors are +-10%"
- note added: "Battery temp current sensing"
- note added: "Battery temp voltage sensing"
- note added: "Battery temperature is monitored with 2 thermistors, should be placed near battery."
- note added: "Buck-Boost"
- note added: "C_L = 12.5 pF"
- note added: "Connection for 5V ICS programmer"
- note added: "LiPo battery connection, 4.2 V max"
- note added: "LiPo charger"
- note added: "RTC"
- note added: "UART bridge"
- note added: "USB ESD protection"
